File: doc/kicad/circuit/circuit.kicad_pcb (KiCad board)
At the start: 2 copper layers, 68.6 x 53.4 mm, 7 parts, among them J1 Analog, J2 Digital, J3 4x4 Button Matrix, J4 Joystick, J5 Pedals, J6 Handbrake, J7 Encoder

Commit message: change the circuit
Parts:
- removed the J3 at (124.7, 73.8)
- added J6: ATmega328P I²C, Connector_PinHeader_2.54mm:PinHeader_1x04_P2.54mm_Vertical_SMD_Pin1Left, F.Cu at (164.7, 92.1)
- added J7.1.1: LCD Socket, Connector_PinSocket_2.54mm:PinSocket_1x16_P2.54mm_Vertical_SMD_Pin1Left, F.Cu at (138.5, 50.1)
- added J7.1.2: PCF8574 LCD Socekt, Connector_PinSocket_2.54mm:PinSocket_1x16_P2.54mm_Vertical_SMD_Pin1Left, F.Cu at (138.5, 58.4)
- added J7.2: PCF8574 I²C, Connector_PinHeader_2.54mm:PinHeader_1x04_P2.54mm_Vertical_SMD_Pin1Left, F.Cu at (155.2, 92.1)
- added R1: 1k, Resistor_SMD:R_0805_2012Metric_Pad1.20x1.40mm_HandSolder, F.Cu at (104.8, 74.2)
- added R2: 1k, Resistor_SMD:R_0805_2012Metric_Pad1.20x1.40mm_HandSolder, F.Cu at (102.8, 74.2)
- J1.1: renamed from J2; footprint Connector_PinSocket_2.54mm:PinSocket_1x17_P2.54mm_Vertical -> Connector_PinSocket_2.54mm:PinSocket_1x17_P2.54mm_Vertical_SMD_Pin1Left
- J1.2: renamed from J1; footprint Connector_PinSocket_2.54mm:PinSocket_1x17_P2.54mm_Vertical -> Connector_PinSocket_2.54mm:PinSocket_1x17_P2.54mm_Vertical_SMD_Pin1Left
- J2: renamed from J6; footprint Connector_PinHeader_2.54mm:PinHeader_1x03_P2.54mm_Vertical -> Connector_PinHeader_2.54mm:PinHeader_1x03_P2.54mm_Vertical_SMD_Pin1Left
- J3: renamed from J7; footprint Connector_PinHeader_2.54mm:PinHeader_1x05_P2.54mm_Vertical -> Connector_PinHeader_2.54mm:PinHeader_1x05_P2.54mm_Vertical_SMD_Pin1Left
- J4, J5: footprint Connector_PinHeader_2.54mm:PinHeader_1x05_P2.54mm_Vertical -> Connector_PinHeader_2.54mm:PinHeader_1x05_P2.54mm_Vertical_SMD_Pin1Left
- moved J5 55.2 mm to (108.8, 52.8)
- moved J4 41.7 mm to (108.8, 59.9)
- moved J1.1 26.0 mm to (124.5, 96.3), turned to 90 degrees
- moved J1.2 21.5 mm to (124.5, 81.1), turned to 90 degrees
- moved J3 9.72 mm to (108.8, 66.8), turned to -90 degrees
- moved J2 4.64 mm to (111.3, 74.3), turned to -90 degrees
Connections:
- J3 pad 1: /Z -> GND
- J3 pad 2: /B -> +5V
- J3 pad 4: +5V -> /B
- J3 pad 5: GND -> /Z
- J4 pad 5: GND -> /*D11

Commit message: start with setup lcd
Parts:
- removed J6: ATmega328P I²C, Connector_PinHeader_2.54mm:PinHeader_1x04_P2.54mm_Vertical_SMD_Pin1Left
- added J1: RJ45, Connector_RJ:RJ45_Molex_0855135013_Vertical, F.Cu at (155.3, 72.4)
- moved J7.2 24.7 mm to (138.1, 74.3), turned to 90 degrees

Commit message: add next i2c button box connector
Parts:
- added J6: RJ45, Connector_RJ:RJ45_Molex_0855135013_Vertical, F.Cu at (157.7, 87.8)
- moved J8 2.60 mm to (157.7, 71.4)
- moved J1.1 1.53 mm to (123.0, 96.3)
- moved J1.2 1.53 mm to (123.0, 81.1)
- moved J7.2 1.47 mm to (139.5, 74.5)
- renumbered J1 to J8

Commit message: finish layout the PCB
Parts:
- added SW1: Reset, Button_Switch_SMD:SW_Push_1P1T_NO_6x6mm_H9.5mm, F.Cu at (126.4, 74.3)
- moved J6 3.22 mm to (157.3, 91.0)
- moved J8 0.57 mm to (157.3, 71.8)
Connections:
- J1.1 pad 13: /~{RESET} -> unconnected-(J1.1-Pin_13-Pad13)
Routing:
- net /*D3/SCL: track 0.00 -> 83.1 mm
- net /D2/SDA: track 0.00 -> 63.3 mm
- net /B: track 0.00 -> 61.5 mm
- net /A0: track 0.00 -> 60.3 mm
- net /A: track 0.00 -> 54.9 mm
- net /A2: track 0.00 -> 49.4 mm
- net /*D11: track 0.00 -> 39.6 mm
- net /A1: track 0.00 -> 37.1 mm
- net /A5: track 0.00 -> 31.5 mm
- net /A4: track 0.00 -> 27.0 mm
- net GND: track 0.00 -> 26.3 mm, vias 0 -> 7
- net /~{RESET}: track 0.00 -> 20.6 mm
- net /A3: track 0.00 -> 15.0 mm
- net Net-(J7.1.1-Pin_9): track 0.00 -> 8.25 mm
- net Net-(J7.1.1-Pin_8): track 0.00 -> 8.25 mm
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- added copper zone on B.Cu, net +5V
- added copper zone on F.Cu, net GND
Other:
- board text added: "github.com/lusmdl/MySimRacingCore"
