File: doc/kicad/circuit/circuit.kicad_sch (KiCad schematic)
At the start: 13 parts, among them J1 Analog, J10 PCF8574 I²C Socket, J2 Digital, J3 4x4 Button Matrix, J4 Joystick, J5 Pedals, J6 Handbrake, J7 Encoder, J8 LCD Socket, J9 PCF8574 LCD Socekt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

Commit message: change the circuit
Parts:
- removed J3: 4x4 Button Matrix, Connector_PinHeader_2.54mm:PinHeader_1x08_P2.54mm_Vertical, symbol Connector:Conn_01x08_Pin
- added J6: ATmega328P I²C, Connector_PinHeader_2.54mm:PinHeader_1x04_P2.54mm_Vertical_SMD_Pin1Left, symbol Connector:Conn_01x04_Pin
- J1.1: renamed from J2; footprint Connector_PinSocket_2.54mm:PinSocket_1x17_P2.54mm_Vertical -> Connector_PinSocket_2.54mm:PinSocket_1x17_P2.54mm_Vertical_SMD_Pin1Left
- J1.2: renamed from J1; footprint Connector_PinSocket_2.54mm:PinSocket_1x17_P2.54mm_Vertical -> Connector_PinSocket_2.54mm:PinSocket_1x17_P2.54mm_Vertical_SMD_Pin1Left
- J2: renamed from J6; footprint Connector_PinHeader_2.54mm:PinHeader_1x03_P2.54mm_Vertical -> Connector_PinHeader_2.54mm:PinHeader_1x03_P2.54mm_Vertical_SMD_Pin1Left
- J3: renamed from J7; footprint Connector_PinHeader_2.54mm:PinHeader_1x05_P2.54mm_Vertical -> Connector_PinHeader_2.54mm:PinHeader_1x05_P2.54mm_Vertical_SMD_Pin1Left
- J4, J5: footprint Connector_PinHeader_2.54mm:PinHeader_1x05_P2.54mm_Vertical -> Connector_PinHeader_2.54mm:PinHeader_1x05_P2.54mm_Vertical_SMD_Pin1Left
- J7.1.1: renamed from J8; footprint (none) -> Connector_PinSocket_2.54mm:PinSocket_1x16_P2.54mm_Vertical_SMD_Pin1Left
- J7.1.2: renamed from J9; footprint (none) -> Connector_PinSocket_2.54mm:PinSocket_1x16_P2.54mm_Vertical_SMD_Pin1Left
- J7.2: renamed from J10; value PCF8574 I²C Socket -> PCF8574 I²C; footprint (none) -> Connector_PinHeader_2.54mm:PinHeader_1x04_P2.54mm_Vertical_SMD_Pin1Left
- R1, R2: footprint (none) -> Resistor_SMD:R_0805_2012Metric_Pad1.20x1.40mm_HandSolder
- U1: footprint Display:LCD-016N002L -> (none); now not fitted; now left out of the parts list
Connections:
- net *D3/SCL: now also J6.4 (Pin_4)
- net +5V: now also J6.2 (Pin_2)
- net D2/SDA: now also J6.3 (Pin_3)
- net GND: now also J6.1 (Pin_1)
Other:
- moved on the sheet: J3, J7.2, R1, R2

Commit message: start with setup lcd
Parts:
- removed J6: ATmega328P I²C, Connector_PinHeader_2.54mm:PinHeader_1x04_P2.54mm_Vertical_SMD_Pin1Left, symbol Connector:Conn_01x04_Pin
- added J1: RJ45, Connector_RJ:RJ45_Molex_0855135013_Vertical, symbol Connector:RJ45
Connections:
- net *D3/SCL: now also J1.7, J1.8
- net +5V: now also J1.3, J1.4
- net D2/SDA: now also J1.5, J1.6
- net GND: now also J1.1, J1.2
Changed lines of the file:
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@@
 	)
 	(junction
-		(at 168.91 121.92)
+		(at 210.82 48.26)
 		(diameter 0)
 		(color 0 0 0 0)
 	)
 	(junction
-		(at 210.82 48.26)
+		(at 210.82 50.8)
 		(diameter 0)
 		(color 0 0 0 0)
 	)
 	(junction
-		(at 210.82 50.8)
+		(at 210.82 38.1)
 		(diameter 0)
 		(color 0 0 0 0)
 	)
 	(junction
-		(at 210.82 38.1)
+		(at 185.42 129.54)
 		(diameter 0)
 		(color 0 0 0 0)
@@
 	)
 	(junction
-		(at 170.18 124.46)
+		(at 168.91 124.46)
 		(diameter 0)
 		(color 0 0 0 0)
@@
 	)
 	(junction
+		(at 170.18 129.54)
+		(diameter 0)
+		(color 0 0 0 0)
+	)
+	(junction
+		(at 185.42 124.46)
+		(diameter 0)
+		(color 0 0 0 0)
+	)
+	(junction
+		(at 185.42 116.84)
+		(diameter 0)
+		(color 0 0 0 0)
+	)
+	(junction
 		(at 210.82 25.4)
 		(diameter 0)
@@
 	)
 	(junction
+		(at 185.42 119.38)
+		(diameter 0)
+		(color 0 0 0 0)
+	)
+	(junction
 		(at 210.82 60.96)
 		(diameter 0)
@@
 	(wire
 		(pts
+			(xy 185.42 114.3) (xy 185.42 116.84)
+		)
+		(stroke
+			(width 0)
+			(type default)
+		)
+	)
+	(wire
+		(pts
 			(xy 260.35 60.96) (xy 237.49 60.96)
 		)
@@
 	(wire
 		(pts
-			(xy 180.34 124.46) (xy 170.18 124.46)
+			(xy 170.18 129.54) (xy 185.42 129.54)
 		)
 		(stroke
@@
 	(wire
 		(pts
+			(xy 185.42 119.38) (xy 185.42 121.92)
+		)
+		(stroke
+			(width 0)
+			(type default)
+		)
+	)
+	(wire
+		(pts
 			(xy 210.82 33.02) (xy 231.14 33.02)
 		)
@@
 	(wire
 		(pts
+			(xy 185.42 129.54) (xy 185.42 132.08)
+		)
+		(stroke
+			(width 0)
+			(type default)
+		)
+	)
+	(wire
+		(pts
 			(xy 62.23 139.7) (xy 127 139.7)
 		)
@@
 	(wire
 		(pts
-			(xy 168.91 121.92) (xy 180.34 121.92)
+			(xy 168.91 124.46) (xy 185.42 124.46)
 		)
 		(stroke
@@
 	(wire
 		(pts
+			(xy 170.18 104.14) (xy 170.18 129.54)
+		)
+		(stroke
+			(width 0)
+			(type default)
+		)
+	)
+	(wire
+		(pts
 			(xy 214.63 149.86) (xy 223.52 149.86)
 		)
@@
 	(wire
 		(pts
+			(xy 185.42 124.46) (xy 185.42 127)
+		)
+		(stroke
+			(width 0)
+			(type default)
+		)
+	)
+	(wire
+		(pts
 			(xy 180.34 99.06) (xy 176.53 99.06)
 		)
@@
 	(wire
 		(pts
+			(xy 168.91 124.46) (xy 168.91 144.78)
+		)
+		(stroke
+			(width 0)
+			(type default)
+		)
+	)
+	(wire
+		(pts
 			(xy 214.63 139.7) (xy 214.63 135.89)
 		)
@@
 	(wire
 		(pts
-			(xy 168.91 101.6) (xy 168.91 121.92)
-		)
-		(stroke
-			(width 0)
-			(type default)
-		)
-	)
-	(wire
-		(pts
 			(xy 232.41 35.56) (xy 210.82 35.56)
 		)
@@
 	(wire
 		(pts
+			(xy 170.18 129.54) (xy 170.18 142.24)
+		)
+		(stroke
+			(width 0)
+			(type default)
+		)
+	)
+	(wire
+		(pts
 			(xy 200.66 33.02) (xy 210.82 33.02)
 		)
@@
 	(wire
 		(pts
-			(xy 180.34 119.38) (xy 172.72 119.38)
+			(xy 172.72 119.38) (xy 185.42 119.38)
 		)
 		(stroke
@@
 	(wire
 		(pts
-			(xy 176.53 116.84) (xy 180.34 116.84)
+			(xy 176.53 116.84) (xy 185.42 116.84)
 		)
 		(stroke
@@
 	(wire
 		(pts
-			(xy 168.91 121.92) (xy 168.91 144.78)
+			(xy 168.91 101.6) (xy 168.91 124.46)
 		)
 		(stroke
@@
 	(wire
 		(pts
-			(xy 170.18 124.46) (xy 170.18 142.24)
-		)
-		(stroke
-			(width 0)
-			(type default)
-		)
-	)
-	(wire
-		(pts
 			(xy 124.46 152.4) (xy 124.46 165.1)
 		)
@@
 	(wire
 		(pts
-			(xy 170.18 104.14) (xy 170.18 124.46)
-		)
-		(stroke
-			(width 0)
-			(type default)
-		)
-	)
-	(wire
-		(pts
 			(xy 176.53 99.06) (xy 176.53 92.71)
 		)
@@
 	)
 	(label "*D3{slash}SCL"
-		(at 172.72 124.46 0)
+		(at 172.72 129.54 0)
 		(fields_autoplaced yes)
 		(effects
@@
 	)
 	(label "D2{slash}SDA"
-		(at 172.72 121.92 0)
+		(at 172.72 124.46 0)
 		(fields_autoplaced yes)
 		(effects
@@
 	)
 	(symbol
-		(lib_id "Connector:Conn_01x04_Pin")
-		(at 185.42 119.38 0)
-		(mirror y)
-		(unit 1)
-		(exclude_from_sim no)
-		(in_bom yes)
-		(on_board yes)
-		(dnp no)
-		(fields_autoplaced yes)
-		(property "Reference" "J6"
-			(at 186.69 119.3799 0)
-			(effects
-				(font
-					(size 1.27 1.27)
-				)
-				(justify right)
-			)
-		)
-		(property "Value" "ATmega328P I²C"
-			(at 186.69 121.9199 0)
-			(effects
-				(font
-					(size 1.27 1.27)
-				)
-				(justify right)
-			)
-		)
-		(property "Footprint" "Connector_PinHeader_2.54mm:PinHeader_1x04_P2.54mm_Vertical_SMD_Pin1Left"
-			(at 185.42 119.38 0)
-			(effects
-				(font
-					(size 1.27 1.27)
-				)
-				(hide yes)
-			)
-		)
-		(property "Datasheet" "~"
-			(at 185.42 119.38 0)
-			(effects
-				(font
-					(size 1.27 1.27)
-				)
-				(hide yes)
-			)
-		)
-		(property "Description" "Generic connector, single row, 01x04, script generated"
-			(at 185.42 119.38 0)
-			(effects
-				(font
-					(size 1.27 1.27)
-				)
-				(hide yes)
-			)
-		)
-		(pin "2"
-		)
-		(pin "3"
-		)
-		(pin "1"
-		)
-		(pin "4"
-		)
-		(instances
-			(project ""
-				(path "/e63e39d7-6ac0-4ffd-8aa3-1841a4541b55"
-					(reference "J6")
-					(unit 1)
-				)
-			)
-		)
-	)
-	(symbol
 		(lib_id "Connector:Conn_01x03_Pin")
 		(at 77.47 132.08 0)
@@
 					(unit 1)
 				)
+			)
+		)
+	)
+	(symbol
+		(lib_id "Connector:RJ45")
+		(at 195.58 121.92 180)
+		(unit 1)
+		(exclude_from_sim no)
+		(in_bom yes)
+		(on_board yes)
+		(dnp no)
+		(fields_autoplaced yes)
+		(property "Reference" "J1"
+			(at 204.47 121.9199 0)
+			(effects
+				(font
+					(size 1.27 1.27)
+				)
+				(justify right)
+			)
+		)
+		(property "Value" "RJ45"
+			(at 204.47 124.4599 0)
+			(effects
+				(font
+					(size 1.27 1.27)
+				)
+				(justify right)
+			)
+		)
+		(property "Footprint" "Connector_RJ:RJ45_Molex_0855135013_Vertical"
+			(at 195.58 122.555 90)
+			(effects
+				(font
+					(size 1.27 1.27)
+				)
+				(hide yes)
+			)
+		)
+		(property "Datasheet" "~"
+			(at 195.58 122.555 90)
+			(effects
+				(font
+					(size 1.27 1.27)
+				)
+				(hide yes)
+			)
+		)
+		(property "Description" "RJ connector, 8P8C (8 positions 8 connected)"
+			(at 195.58 121.92 0)
+			(effects
+				(font
+					(size 1.27 1.27)
+				)
+				(hide yes)
+			)
+		)
+		(pin "4"
+		)
+		(pin "6"
+		)
+		(pin "2"
+		)
+		(pin "3"
+		)
+		(pin "8"
+		)
+		(pin "7"
+		)
+		(pin "5"
+		)
+		(pin "1"
+		)
+		(instances
+			(project ""
+				(path "/e63e39d7-6ac0-4ffd-8aa3-1841a4541b55"
+					(reference "J1")
+					(unit 1)
+				)

Commit message: add next i2c button box connector
Parts:
- added J6: RJ45, Connector_RJ:RJ45_Molex_0855135013_Vertical, symbol Connector:RJ45
- renumbered J1 to J8
Connections:
- net *D3/SCL: now also J6.7, J6.8
- net +5V: now also J6.3, J6.4
- net D2/SDA: now also J6.5, J6.6
- net GND: now also J6.1, J6.2

Commit message: finish layout the PCB
Parts:
- added SW1: Reset, Button_Switch_SMD:SW_Push_1P1T_NO_6x6mm_H9.5mm, symbol Switch:SW_Push
Connections:
- net GND: now also SW1.1
- net ~{RESET}: now also SW1.2; no longer J1.1.13 (Pin_13)
Changed lines of the file:
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@@
+	)
+	(junction
+		(at 124.46 152.4)
+		(diameter 0)
+		(color 0 0 0 0)
 	)
 	(junction
@@
 	(wire
 		(pts
+			(xy 95.25 152.4) (xy 124.46 152.4)
+		)
+		(stroke
+			(width 0)
+			(type default)
+		)
+	)
+	(wire
+		(pts
 			(xy 200.66 58.42) (xy 210.82 58.42)
 		)
@@
 	(wire
 		(pts
+			(xy 95.25 149.86) (xy 95.25 152.4)
+		)
+		(stroke
+			(width 0)
+			(type default)
+		)
+	)
+	(wire
+		(pts
 			(xy 185.42 109.22) (xy 218.44 109.22)
 		)
@@
 	(wire
 		(pts
+			(xy 105.41 149.86) (xy 127 149.86)
+		)
+		(stroke
+			(width 0)
+			(type solid)
+		)
+	)
+	(wire
+		(pts
 			(xy 147.32 139.7) (xy 162.56 139.7)
 		)
@@
 	(wire
 		(pts
-			(xy 111.76 149.86) (xy 127 149.86)
-		)
-		(stroke
-			(width 0)
-			(type solid)
-		)
-	)
-	(wire
-		(pts
 			(xy 182.88 124.46) (xy 182.88 106.68)
 		)
@@
 		(pts
 			(xy 99.06 127) (xy 127 127)
-		)
-		(stroke
-			(width 0)
-			(type solid)
-		)
-	)
-	(wire
-		(pts
-			(xy 147.32 149.86) (xy 162.56 149.86)
 		)
 		(stroke
@@
 			)
 			(justify left bottom)
-		)
-	)
-	(label "~{RESET}"
-		(at 162.56 149.86 180)
-		(fields_autoplaced yes)
-		(effects
-			(font
-				(size 1.27 1.27)
-			)
-			(justify right bottom)
 		)
 	)
@@
 					(unit 1)
 				)
+			)
+		)
+	)
+	(symbol
+		(lib_id "Switch:SW_Push")
+		(at 100.33 149.86 0)
+		(unit 1)
+		(exclude_from_sim no)
+		(in_bom yes)
+		(on_board yes)
+		(dnp no)
+		(property "Reference" "SW1"
+			(at 92.456 147.066 0)
+			(effects
+				(font
+					(size 1.27 1.27)
+				)
+			)
+		)
+		(property "Value" "Reset"
+			(at 100.33 144.78 0)
+			(effects
+				(font
+					(size 1.27 1.27)
+				)
+			)
+		)
+		(property "Footprint" "Button_Switch_SMD:SW_Push_1P1T_NO_6x6mm_H9.5mm"
+			(at 100.33 144.78 0)
+			(effects
+				(font
+					(size 1.27 1.27)
+				)
+				(hide yes)
+			)
+		)
+		(property "Datasheet" "~"
+			(at 100.33 144.78 0)
+			(effects
+				(font
+					(size 1.27 1.27)
+				)
+				(hide yes)
+			)
+		)
+		(property "Description" "Push button switch, generic, two pins"
+			(at 100.33 149.86 0)
+			(effects
+				(font
+					(size 1.27 1.27)
+				)
+				(hide yes)
+			)
+		)
+		(pin "1"
+		)
+		(pin "2"
+		)
+		(instances
+			(project ""
+				(path "/e63e39d7-6ac0-4ffd-8aa3-1841a4541b55"
+					(reference "SW1")
+					(unit 1)
+				)
